File: 12-input-pulse-counter/12input.brd (EAGLE design)
At the start: 65 parts, among them CN1 1X4-3.5MM, CN2 1X4-3.5MM, CN3 1X4-3.5MM, U1 ATMEGA168, U2 ATMEGA168

Commit message: Updated relay-unit with atmega328 and rfm12/69
Parts:
- removed JP2, JP3: (no value), adafruit:1X06
- removed RFM12B: RFM12B, JeeLabs:RFM12B
- removed SJ5: Wiznet SS, jumper:SJ_2W
- removed U1: ATMEGA168, SparkFun:TQFP32-08
- added C1, C11: 22pF, resistor:C0603
- added C10, C9: 100nF, rcl:C0603
- added C16, C19: 20pF, rcl:C0603
- added C3: 0.1uF, rcl:C0603
- added C6, C8: 0.1uF, resistor:C0603
- added J$1: SMA_EDGE, SparkFun-Connectors:SMA-EDGE
- added Q1: 16Mhz, adafruit:HC49UP
- added R38: 10K, adafruit:R0603
- added R39: 100K, rcl:R0603
- added U$14: RFM12B, JeeParts:RFM12B
- added U1_MLF: ATMEGA168MLF, SparkFun-DigitalIC:MLF32
- added U1_TQFP: ATMEGA328P, SparkFun-DigitalIC:TQFP32-08
- ISP: value AVR_SPI_PRG_6PTH -> 2x3
- JP1: value (none) -> FTDI; device SparkFun:1X02 -> SparkFun:FTDI_BASIC
- moved ANT1 109.5 mm to (1.91, -39.4)
- moved ISP 97.2 mm to (17.8, -21.6), turned to 0 degrees
- moved JP1 96.2 mm to (17.8, -29.2)
Connections:
- removed net DIG10: SJ5.1
- removed net MASTER_D10: RFM12B.SEL, U1.14
- removed net MASTER_D11/MOSI: RFM12B.SDI, U1.15
- removed net MASTER_D12/MISO: RFM12B.SDO, U1.16
- removed net MASTER_D13/SCK: RFM12B.SCK, U1.17
- removed net MASTER_D2: RFM12B.IRQ, U1.32
- removed net MISO: JP3.6
- removed net MOSI: JP2.3
- removed net RST: JP3.5
- removed net SCK: JP2.4
- removed net SS: JP2.5, SJ5.2, SJ5.3
- new net ADC0: U1_MLF.23, U1_TQFP.23
- new net ADC1: U1_MLF.24, U1_TQFP.24
- new net ADC2: U1_MLF.25, U1_TQFP.25
- new net ADC3: U1_MLF.26, U1_TQFP.26
- new net ADC4: U1_MLF.27, U1_TQFP.27
- new net ADC5: U1_MLF.28, U1_TQFP.28
- new net DIG1: C16.1, C19.1, U$14.ANT
- new net N$1: C1.1, Q1.2, U1_MLF.7, U1_TQFP.7
- new net N$20: C8.1, U1_MLF.20, U1_TQFP.20
- new net N$24: C19.2, J$1.SIG
- new net N$4: C11.1, Q1.1, U1_MLF.8, U1_TQFP.8
- new net N$5: ANT1.1, C16.2
- new net N$8: C9.2, JP1.DTR
- net +3V3: no longer JP1.2, RFM12B.VDD
- net +5V: now also JP1.VCC; no longer ISP.2, JP1.1
- net 3.3V: now also C10.1, C3.1, C6.1, ISP.2, R38.2, R39.2, U$14.VDD, U1_MLF.18, U1_MLF.4, U1_MLF.6, U1_TQFP.18, U1_TQFP.4, U1_TQFP.6; no longer JP3.2, JP3.3
- net A6: now also U1_MLF.19, U1_TQFP.19
- net A7: now also U1_MLF.22, U1_TQFP.22
- net D0/RX: now also JP1.TXO, U1_MLF.30, U1_TQFP.30
- net D1/TX: now also JP1.RXI, U1_MLF.31, U1_TQFP.31
- net D10: now also R39.1, U$14.SEL, U1_MLF.14, U1_TQFP.14
- net D11/MOSI: now also U$14.SDI, U1_MLF.15, U1_TQFP.15
- net D12/MISO: now also U$14.SDO, U1_MLF.16, U1_TQFP.16
- net D13/SCK: now also U$14.SCK, U1_MLF.17, U1_TQFP.17
- net D2: now also U$14.IRQ, U1_MLF.32, U1_TQFP.32
- net D3: now also U1_MLF.1, U1_TQFP.1
- net D4: now also U1_MLF.2, U1_TQFP.2
- net D5: now also U1_MLF.9, U1_TQFP.9
- net D6: now also U1_MLF.10, U1_TQFP.10
- net D7: now also U1_MLF.11, U1_TQFP.11
- net D8: now also U1_MLF.12, U1_TQFP.12
- net D9: now also U1_MLF.13, U1_TQFP.13
- net GND: now also C1.2, C10.2, C11.2, C3.2, C6.2, C8.2, J$1.GND@0, J$1.GND@1, J$1.GND@2, J$1.GND@3, JP1.GND, U$14.GND, U$14.P$12, U1_MLF.21, U1_MLF.3, U1_MLF.5, U1_TQFP.21, U1_TQFP.3, U1_TQFP.5; no longer JP2.1, JP2.2, JP3.1, RFM12B.GND
- net N$6: now also JP1.CTS; no longer ANT1.1, RFM12B.ANT
- net RESET: now also C9.1, R38.1, U1_MLF.29, U1_TQFP.29
