File: 12-input-pulse-counter/12input.sch (EAGLE design)
At the start: 64 parts, among them CN1 1X4-3.5MM, CN2 1X4-3.5MM, CN3 1X4-3.5MM, U1 ATMEGA168, U2 ATMEGA168

Commit message: Updated relay-unit with atmega328 and rfm12/69
Parts:
- removed JP2, JP3: (no value), adafruit:PINHD-1X6
- removed RFM12B: RFM12B, JeeLabs:RFM12B
- removed SJ5: Wiznet SS, jumper:SJ2WW
- removed U1: ATMEGA168, SparkFun:ATMEGA168
- added C1, C11: 22pF, resistor:C-EUC0603
- added C10, C9: 100nF, rcl:C-EUC0603
- added C16, C19: 20pF, rcl:C-EUC0603
- added C3: 0.1uF, rcl:C-EUC0603
- added C6, C8: 0.1uF, resistor:C-EUC0603
- added J$1: SMA_EDGE, SparkFun-Connectors:SMA_EDGE
- added Q1: 16Mhz, adafruit:CRYSTALHC49UP
- added R38: 10K, adafruit:R-US_R0603
- added R39: 100K, rcl:R-EU_R0603
- added U$14: RFM12B, JeeParts:RFM12B
- added U1_MLF: ATMEGA168MLF, SparkFun-DigitalIC:ATMEGA168MLF
- added U1_TQFP: ATMEGA328P, SparkFun-DigitalIC:ATMEGA328_SMT
- ISP: value AVR_SPI_PRG_6PTH -> 2x3
- JP1: value (none) -> FTDI; device SparkFun:JUMPER-2PTH -> SparkFun:FTDI_BASICPTH
Connections:
- removed net DIG10: SJ5.1
- removed net MASTER_D10: RFM12B.SEL, U1.PB2(SS/OC1B)
- removed net MASTER_D11/MOSI: RFM12B.SDI, U1.PB3(MOSI/OC2)
- removed net MASTER_D12/MISO: RFM12B.SDO, U1.PB4(MISO)
- removed net MASTER_D13/SCK: RFM12B.SCK, U1.PB5(SCK)
- removed net MASTER_D2: RFM12B.IRQ, U1.PD2(INT0)
- removed net MISO: JP3.6
- removed net MOSI: JP2.3
- removed net RST: JP3.5
- removed net SCK: JP2.4
- removed net SS: JP2.5, SJ5.2, SJ5.3
- new net ADC0: U1_MLF.PC0(ADC0), U1_TQFP.PC0(ADC0)
- new net ADC1: U1_MLF.PC1(ADC1), U1_TQFP.PC1(ADC1)
- new net ADC2: U1_MLF.PC2(ADC2), U1_TQFP.PC2(ADC2)
- new net ADC3: U1_MLF.PC3(ADC3), U1_TQFP.PC3(ADC3)
- new net ADC4: U1_MLF.PC4(ADC4/SDA), U1_TQFP.PC4(ADC4/SDA)
- new net ADC5: U1_MLF.PC5(ADC5/SCL), U1_TQFP.PC5(ADC5/SCL)
- new net DIG1: C16.1, C19.1, U$14.ANT
- new net N$1: C1.1, Q1.2, U1_MLF.PB6(XTAL1/TOSC1), U1_TQFP.PB6(XTAL1/TOSC1)
- new net N$20: C8.1, U1_MLF.AREF, U1_TQFP.AREF
- new net N$24: C19.2, J$1.SIGNAL
- new net N$4: C11.1, Q1.1, U1_MLF.PB7(XTAL2/TOSC2), U1_TQFP.PB7(XTAL2/TOSC2)
- new net N$5: ANT1.1, C16.2
- new net N$8: C9.2, JP1.1
- net +3V3: no longer JP1.2, RFM12B.VCC
- net +5V: now also JP1.4; no longer ISP.2, JP1.1
- net 3.3V: now also C10.1, C3.1, C6.1, ISP.2, R38.2, R39.2, U$14.VCC, U1_MLF.AVCC, U1_MLF.VCC@1, U1_MLF.VCC@2, U1_TQFP.AVCC, U1_TQFP.VCC@1, U1_TQFP.VCC@2; no longer JP3.2, JP3.3
- net A6: now also U1_MLF.ADC6, U1_TQFP.ADC6
- net A7: now also U1_MLF.ADC7, U1_TQFP.ADC7
- net D0/RX: now also JP1.3, U1_MLF.PD0(RXD), U1_TQFP.PD0(RXD)
- net D1/TX: now also JP1.2, U1_MLF.PD1(TXD), U1_TQFP.PD1(TXD)
- net D10: now also R39.1, U$14.SEL, U1_MLF.PB2(SS/OC1B), U1_TQFP.PB2(SS/OC1B)
- net D11/MOSI: now also U$14.SDI, U1_MLF.PB3(MOSI/OC2), U1_TQFP.PB3(MOSI/OC2)
- net D12/MISO: now also U$14.SDO, U1_MLF.PB4(MISO), U1_TQFP.PB4(MISO)
- net D13/SCK: now also U$14.SCK, U1_MLF.PB5(SCK), U1_TQFP.PB5(SCK)
- net D2: now also U$14.IRQ, U1_MLF.PD2(INT0), U1_TQFP.PD2(INT0)
- net D3: now also U1_MLF.PD3(INT1), U1_TQFP.PD3(INT1)
- net D4: now also U1_MLF.PD4(XCK/T0), U1_TQFP.PD4(XCK/T0)
- net D5: now also U1_MLF.PD5(T1), U1_TQFP.PD5(T1)
- net D6: now also U1_MLF.PD6(AIN0), U1_TQFP.PD6(AIN0)
- net D7: now also U1_MLF.PD7(AIN1), U1_TQFP.PD7(AIN1)
- net D8: now also U1_MLF.PB0(ICP), U1_TQFP.PB0(ICP)
- net D9: now also U1_MLF.PB1(OC1A), U1_TQFP.PB1(OC1A)
- net GND: now also C1.2, C10.2, C11.2, C3.2, C6.2, C8.2, J$1.GND@0, J$1.GND@1, J$1.GND@2, J$1.GND@3, JP1.6, U$14.GND, U1_MLF.AGND, U1_MLF.GND@1, U1_MLF.GND@2, U1_TQFP.AGND, U1_TQFP.GND@1, U1_TQFP.GND@2; no longer JP2.1, JP2.2, JP3.1, RFM12B.GND
- net N$6: now also JP1.5; no longer ANT1.1, RFM12B.ANT
- net RESET: now also C9.1, R38.1, U1_MLF.PC6(/RESET), U1_TQFP.PC6(/RESET)
Other:
- note added: "ATmega328"
- note added: "RFM12B RFM1269CW"
- note added: "UART & ISP"
- note removed: "Wiznet SS Select line default to SS (DIG17)"
- note removed: "Wiznet W5200 820io"
- moved on the sheet: ANT1, ISP
