File: RFM2Pi/board/KiCad_RFM12Pi V2.7/KiCad_test.kicad_pcb (KiCad board)
At the start: 2 copper layers, 30 x 30 mm, 14 parts, among them CON1 AVR-ISP-6, IC1 ATMEGA328P-A, IC2 ATMEGA328P-A, P1 CONN_02X05_RasPi_GPIO, P2 CONN_01X01, U1 RFM12

Commit message: RFM12Pi V2.7 revision compleate using kicad
Parts:
- added ?: Symbol_OSHW-Logo_SilkScreen_07Jul2012, Symbols:Symbol_OSHW-Logo_SilkScreen, B.Cu at (146.1, 97.7)
- renumbered P2 to ANT, D1 to LED
Connections:
- IC2 pad 33: (no net) -> GND
Routing:
- net GND: track 100.7 -> 131.1 mm, vias 1 -> 5
- net +3.3V: track 118.2 -> 119.6 mm
- net (no net): track 0.00 -> 0.18 mm, vias 0 -> 7
- added copper zone on B.Cu, net GND
- added copper zone on F.Cu, net GND
Other:
- board text added: "+"
- board text added: "-"
- board text added: "433Mhz 868Mhz"
- board text added: "OpenEnergyMonitor.org RFM12Pi V2.7 Oct14"
- board text removed: "OpenEnergyMonitor.org RFM12Pi V2.7"
