File: RFM2Pi/board/KiCad_RFM12Pi V2.7/KiCad_test.sch (KiCad schematic (older format))
At the start: 14 parts, among them CON1 AVR-ISP-6, IC1 ATMEGA328P-A, IC2 ATMEGA328P-A, P1 CONN_02X05_RasPi_GPIO, P2 CONN_01X01, U1 RFM12

Commit message: update kicad and remove rfm12ppi frmware, see openenergymonitor/rfm12pi repo for latest firmware
Parts:
- P2: footprint Connect:PINTST -> ant:PINTST
- R1, R2, R3: footprint Resistors_SMD:R_0603 -> SMD_Packages:SMD-0603
Changed lines of the file:
@@
 F 0 "R1" V 6980 1900 40  0000 C CNN
 F 1 "220R" V 6907 1901 40  0000 C CNN
-F 2 "Resistors_SMD:R_0603" V 6830 1900 30  0001 C CNN
+F 2 "SMD_Packages:SMD-0603" V 6830 1900 30  0001 C CNN
 F 3 "" H 6900 1900 30  0000 C CNN
 	1    6900 1900
@@
 F 0 "R2" V 9030 3750 40  0000 C CNN
 F 1 "100K" V 8957 3751 40  0000 C CNN
-F 2 "Resistors_SMD:R_0603" V 8880 3750 30  0001 C CNN
+F 2 "SMD_Packages:SMD-0603" V 8880 3750 30  0001 C CNN
 F 3 "" H 8950 3750 30  0000 C CNN
 	1    8950 3750
@@
 F 0 "R3" V 6280 2950 40  0000 C CNN
 F 1 "10K" V 6207 2951 40  0000 C CNN
-F 2 "Resistors_SMD:R_0603" V 6130 2950 30  0001 C CNN
+F 2 "SMD_Packages:SMD-0603" V 6130 2950 30  0001 C CNN
 F 3 "" H 6200 2950 30  0000 C CNN
 	1    6200 2950
@@
 F 0 "P2" H 9600 4850 50  0000 C CNN
 F 1 "CONN_01X01" V 9700 4750 50  0000 C CNN
-F 2 "Connect:PINTST" H 9600 4750 60  0001 C CNN
+F 2 "ant:PINTST" H 9600 4750 60  0001 C CNN
 F 3 "" H 9600 4750 60  0000 C CNN
 	1    9600 4750
