File: RFM2Pi/board/RFM69Pi_V3.1/RFM69Pi_V3.1.sch (EAGLE design)
At the start: 18 parts, among them IC1 ATMEGA168

Commit message: add RFM12Pi V3.1
Parts:
- removed ANT: (no value), JeeLabs:1,6/0,8
- added ANT1: (no value), discrete:ANTENNA
- R4: value 220R -> 1K
- renumbered RASPBERRY-PI to GPIO_1
Connections:
- net N$6: now also ANT1.1; no longer ANT.P
Changed lines of the file:
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@@
 <?xml version="1.0" encoding="utf-8"?>
 <!DOCTYPE eagle SYSTEM "eagle.dtd">
-<eagle version="7.0.0">
+<eagle version="7.2.0">
 <drawing>
 <settings>
@@
 <classes>
 <class number="0" name="default" width="0.2032" drill="0.2032">
-<clearance class="0" value="0.2032"/>
+<clearance class="0" value="0.205"/>
 </class>
 <class number="1" name="power" width="0.254" drill="0.254">
+<clearance class="0" value="0.205"/>
 <clearance class="1" value="0.254"/>
 </class>
@@
 <part name="+3V2" library="supply1" deviceset="+3V3" device=""/>
 <part name="GND2" library="supply1" deviceset="GND" device=""/>
-<part name="ANT" library="JeeLabs" deviceset="1,6/0,8" device=""/>
-<part name="RASPBERRY-PI" library="con-lsta" deviceset="FE05-2" device=""/>
+<part name="GPIO_1" library="con-lsta" deviceset="FE05-2" device=""/>
 <part name="+3V8" library="supply1" deviceset="+3V3" device=""/>
 <part name="GND5" library="supply1" deviceset="GND" device=""/>
 <part name="LED1" library="led" deviceset="LED" device="SML0603"/>
-<part name="R4" library="adafruit" deviceset="R-US_" device="R0603" value="220R"/>
+<part name="R4" library="adafruit" deviceset="R-US_" device="R0603" value="1K"/>
 <part name="GND8" library="supply1" deviceset="GND" device=""/>
 <part name="C4" library="rcl" deviceset="C-EU" device="C0603" value="0.1uF"/>
@@
 <part name="R2" library="adafruit" deviceset="R-US_" device="R0603" value="10K"/>
 <part name="C3" library="rcl" deviceset="C-EU" device="C0603" value="10uF"/>
+<part name="ANT1" library="discrete" deviceset="ANTENNA" device=""/>
 </parts>
 <sheets>
@@
 <instance part="+3V2" gate="G$1" x="7.62" y="91.44"/>
 <instance part="GND2" gate="1" x="7.62" y="35.56"/>
-<instance part="ANT" gate="P" x="25.4" y="53.34" rot="R180"/>
-<instance part="RASPBERRY-PI" gate="G$1" x="-66.04" y="116.84"/>
+<instance part="GPIO_1" gate="G$1" x="-66.04" y="116.84"/>
 <instance part="+3V8" gate="G$1" x="-48.26" y="114.3"/>
 <instance part="GND5" gate="1" x="-81.28" y="114.3"/>
@@
 <instance part="R2" gate="G$1" x="-10.16" y="71.12" rot="R90"/>
 <instance part="C3" gate="G$1" x="33.02" y="58.42" rot="R180"/>
+<instance part="ANT1" gate="A" x="22.86" y="48.26" rot="R180"/>
 </instances>
 <busses>
@@
 </segment>
 <segment>
-<pinref part="RASPBERRY-PI" gate="G$1" pin="2"/>
+<pinref part="GPIO_1" gate="G$1" pin="2"/>
 <wire x1="-58.42" y1="111.76" x2="-48.26" y2="111.76" width="0.1524" layer="91"/>
 <pinref part="+3V8" gate="G$1" pin="+3V3"/>
@@
 </segment>
 <segment>
-<pinref part="RASPBERRY-PI" gate="G$1" pin="5"/>
+<pinref part="GPIO_1" gate="G$1" pin="5"/>
 <wire x1="-73.66" y1="116.84" x2="-81.28" y2="116.84" width="0.1524" layer="91"/>
 <pinref part="GND5" gate="1" pin="GND"/>
@@
 </segment>
 <segment>
-<pinref part="RASPBERRY-PI" gate="G$1" pin="10"/>
+<pinref part="GPIO_1" gate="G$1" pin="10"/>
 <wire x1="-58.42" y1="121.92" x2="-30.48" y2="121.92" width="0.1524" layer="91"/>
 <wire x1="-30.48" y1="121.92" x2="-30.48" y2="116.84" width="0.1524" layer="91"/>
@@
 <segment>
 <pinref part="RFM12B-RFM69CW" gate="G$1" pin="ANT"/>
-<pinref part="ANT" gate="P" pin="P"/>
 <wire x1="20.32" y1="53.34" x2="22.86" y2="53.34" width="0.1524" layer="91"/>
+<pinref part="ANT1" gate="A" pin="1"/>
 </segment>
 </net>
@@
 </segment>
 <segment>
-<pinref part="RASPBERRY-PI" gate="G$1" pin="9"/>
+<pinref part="GPIO_1" gate="G$1" pin="9"/>
 <wire x1="-73.66" y1="121.92" x2="-81.28" y2="121.92" width="0.1524" layer="91"/>
 <label x="-86.36" y="121.92" size="1.778" layer="95"/>
@@
 </segment>
 <segment>
-<pinref part="RASPBERRY-PI" gate="G$1" pin="7"/>
+<pinref part="GPIO_1" gate="G$1" pin="7"/>
 <wire x1="-73.66" y1="119.38" x2="-81.28" y2="119.38" width="0.1524" layer="91"/>
 <label x="-86.36" y="119.38" size="1.778" layer="95"/>
@@
 </segment>
 <segment>
-<pinref part="RASPBERRY-PI" gate="G$1" pin="8"/>
+<pinref part="GPIO_1" gate="G$1" pin="8"/>
 <wire x1="-58.42" y1="119.38" x2="-48.26" y2="119.38" width="0.1524" layer="91"/>
 <label x="-48.26" y="119.38" size="1.778" layer="95"/>
