File: emonTH/emonTH_V2_0/emonTH V2.0.0.brd (EAGLE design)
At the start: 54.1 x 64 mm, 47 parts, among them J1 1X2-3.5MM, J2 1X2-3.5MM, J3 1X2-3.5MM, Q1 16Mhz, Q2 DS18B20, U1 LTC3525ESC6-3.3TRMPBF, U1_MLF ATMEGA168MLF, U1_TQFP ATMEGA328P, U2 SI7021

Commit message: add emonth v2.0.1 led footprint update
Parts:
- LED: value Green -> (none); device adafruit:CHIP-LED0805 -> adafruit:CHIPLED-0603-TTW
- moved LED 1.30 mm to (31.5, 2.54)
Routing:
- net GND: track 289.9 -> 288.0 mm
- net N$1: track 5.72 -> 7.57 mm
Other:
- board text added: "emonTH V2.0.1 Aug 2016 Temperature & Humidity Node"
- board text removed: "emonTH V2.0.0 Aug 2016 Temperature & Humidity Node"
